File: KiCad/GPIO_to_24V/GPIO_to_24V.sch (KiCad schematic (older format))
At the start: 14 parts, among them U1 ! 4N33 !, U1 TLP627-4, U2 ! 4N33 !, U3 ! 4N33 !, U4 ! 4N33 !

Commit message: Schematics
Parts:
- removed D? (x3): 1N4148, Diode_THT:D_DO-35_SOD27_P7.62mm_Horizontal, symbol Diode:1N4148
- removed R2, R3, R4: R, symbol Device:R
- removed U2, U3, U4: ! 4N33 !, Package_DIP:DIP-6_W7.62mm, symbol Isolator:4N28
Changed lines of the file:
@@
 Wire Wire Line
 	5250 1200 5450 1200
-Wire Wire Line
-	5250 1950 5450 1950
-Wire Wire Line
-	5250 2700 5450 2700
-Wire Wire Line
-	5250 3450 5450 3450
 $Comp
 L power:GND #PWR?
@@
 F 3 "" H 5450 1400 50  0001 C CNN
 	1    5450 1400
-	0    1    1    0
-$EndComp
-$Comp
-L power:GND #PWR?
-U 1 1 648AD733
-P 5450 2150
-F 0 "#PWR?" H 5450 1900 50  0001 C CNN
-F 1 "GND" V 5455 2022 50  0000 R CNN
-F 2 "" H 5450 2150 50  0001 C CNN
-F 3 "" H 5450 2150 50  0001 C CNN
-	1    5450 2150
-	0    1    1    0
-$EndComp
-$Comp
-L power:GND #PWR?
-U 1 1 648AD739
-P 5450 2900
-F 0 "#PWR?" H 5450 2650 50  0001 C CNN
-F 1 "GND" V 5455 2772 50  0000 R CNN
-F 2 "" H 5450 2900 50  0001 C CNN
-F 3 "" H 5450 2900 50  0001 C CNN
-	1    5450 2900
-	0    1    1    0
-$EndComp
-$Comp
-L power:GND #PWR?
-U 1 1 648AD73F
-P 5450 3650
-F 0 "#PWR?" H 5450 3400 50  0001 C CNN
-F 1 "GND" V 5455 3522 50  0000 R CNN
-F 2 "" H 5450 3650 50  0001 C CNN
-F 3 "" H 5450 3650 50  0001 C CNN
-	1    5450 3650
 	0    1    1    0
 $EndComp
@@
 	1    0    0    -1
 $EndComp
-$Comp
-L power:GND1 #PWR?
-U 1 1 648AD74B
-P 6250 2350
-F 0 "#PWR?" H 6250 2100 50  0001 C CNN
-F 1 "GND1" H 6255 2177 50  0000 C CNN
-F 2 "" H 6250 2350 50  0001 C CNN
-F 3 "" H 6250 2350 50  0001 C CNN
-	1    6250 2350
-	1    0    0    -1
-$EndComp
-$Comp
-L power:GND1 #PWR?
-U 1 1 648AD751
-P 6250 3100
-F 0 "#PWR?" H 6250 2850 50  0001 C CNN
-F 1 "GND1" H 6255 2927 50  0000 C CNN
-F 2 "" H 6250 3100 50  0001 C CNN
-F 3 "" H 6250 3100 50  0001 C CNN
-	1    6250 3100
-	1    0    0    -1
-$EndComp
-$Comp
-L power:GND1 #PWR?
-U 1 1 648AD757
-P 6250 3850
-F 0 "#PWR?" H 6250 3600 50  0001 C CNN
-F 1 "GND1" H 6255 3677 50  0000 C CNN
-F 2 "" H 6250 3850 50  0001 C CNN
-F 3 "" H 6250 3850 50  0001 C CNN
-	1    6250 3850
-	1    0    0    -1
-$EndComp
 Text GLabel 4850 1200 0    50   Input ~ 0
 IN-1
-Text GLabel 4850 1950 0    50   Input ~ 0
-IN-2
-Text GLabel 4850 2700 0    50   Input ~ 0
-IN-3
-Text GLabel 4850 3450 0    50   Input ~ 0
-IN-4
 Text GLabel 6550 1300 2    50   Output ~ 0
 Out-1
-Text GLabel 6550 2050 2    50   Output ~ 0
-Out-2
-Text GLabel 6550 2800 2    50   Output ~ 0
-Out-3
-Text GLabel 6550 3550 2    50   Output ~ 0
-Out-4
 Wire Wire Line
 	4850 1200 4950 1200
-Wire Wire Line
-	4850 1950 4950 1950
-Wire Wire Line
-	4850 2700 4950 2700
-Wire Wire Line
-	4850 3450 4950 3450
 $Comp
 L Isolator:4N28 U1
@@
 F 3 "https://www.vishay.com/docs/83725/4n25.pdf" H 5750 1300 50  0001 L CNN
 	1    5750 1300
-	1    0    0    -1
-$EndComp
-$Comp
-L Isolator:4N28 U2
-U 1 1 648B0EB6
-P 5750 2050
-F 0 "U2" H 5750 2375 50  0000 C CNN
-F 1 "! 4N33 !" H 5750 2284 50  0000 C CNN
-F 2 "Package_DIP:DIP-6_W7.62mm" H 5550 1850 50  0001 L CIN
-F 3 "https://www.vishay.com/docs/83725/4n25.pdf" H 5750 2050 50  0001 L CNN
-	1    5750 2050
-	1    0    0    -1
-$EndComp
-$Comp
-L Isolator:4N28 U3
-U 1 1 648B20C6
-P 5750 2800
-F 0 "U3" H 5750 3125 50  0000 C CNN
-F 1 "! 4N33 !" H 5750 3034 50  0000 C CNN
-F 2 "Package_DIP:DIP-6_W7.62mm" H 5550 2600 50  0001 L CIN
-F 3 "https://www.vishay.com/docs/83725/4n25.pdf" H 5750 2800 50  0001 L CNN
-	1    5750 2800
-	1    0    0    -1
-$EndComp
-$Comp
-L Isolator:4N28 U4
-U 1 1 648B3317
-P 5750 3550
-F 0 "U4" H 5750 3875 50  0000 C CNN
-F 1 "! 4N33 !" H 5750 3784 50  0000 C CNN
-F 2 "Package_DIP:DIP-6_W7.62mm" H 5550 3350 50  0001 L CIN
-F 3 "https://www.vishay.com/docs/83725/4n25.pdf" H 5750 3550 50  0001 L CNN
-	1    5750 3550
 	1    0    0    -1
 $EndComp
@@
 	0    1    1    0
 $EndComp
-$Comp
-L Diode:1N4148 D?
-U 1 1 648D24F9
-P 6250 2200
-F 0 "D?" V 6204 2280 50  0000 L CNN
-F 1 "1N4148" V 6295 2280 50  0000 L CNN
-F 2 "Diode_THT:D_DO-35_SOD27_P7.62mm_Horizontal" H 6250 2025 50  0001 C CNN
-F 3 "https://assets.nexperia.com/documents/data-sheet/1N4148_1N4448.pdf" H 6250 2200 50  0001 C CNN
-	1    6250 2200
-	0    1    1    0
-$EndComp
-$Comp
-L Diode:1N4148 D?
-U 1 1 648D3490
-P 6250 2950
-F 0 "D?" V 6204 3030 50  0000 L CNN
-F 1 "1N4148" V 6295 3030 50  0000 L CNN
-F 2 "Diode_THT:D_DO-35_SOD27_P7.62mm_Horizontal" H 6250 2775 50  0001 C CNN
-F 3 "https://assets.nexperia.com/documents/data-sheet/1N4148_1N4448.pdf" H 6250 2950 50  0001 C CNN
-	1    6250 2950
-	0    1    1    0
-$EndComp
-$Comp
-L Diode:1N4148 D?
-U 1 1 648D44FC
-P 6250 3700
-F 0 "D?" V 6204 3780 50  0000 L CNN
-F 1 "1N4148" V 6295 3780 50  0000 L CNN
-F 2 "Diode_THT:D_DO-35_SOD27_P7.62mm_Horizontal" H 6250 3525 50  0001 C CNN
-F 3 "https://assets.nexperia.com/documents/data-sheet/1N4148_1N4448.pdf" H 6250 3700 50  0001 C CNN
-	1    6250 3700
-	0    1    1    0
-$EndComp
-Wire Wire Line
-	6050 2350 6050 2150
 Wire Wire Line
 	6050 1600 6050 1400
 Wire Wire Line
-	6050 3100 6050 2900
-Wire Wire Line
-	6050 3850 6050 3650
-Wire Wire Line
 	6250 1300 6550 1300
-Wire Wire Line
-	6250 2050 6550 2050
-Wire Wire Line
-	6250 2800 6550 2800
-Wire Wire Line
-	6250 3550 6550 3550
 Wire Wire Line
 	6050 1300 6250 1300
@@
 	6050 1600 6250 1600
 Connection ~ 6250 1600
-Wire Wire Line
-	6050 2050 6250 2050
-Connection ~ 6250 2050
-Wire Wire Line
-	6050 2350 6250 2350
-Connection ~ 6250 2350
-Wire Wire Line
-	6050 2800 6250 2800
-Connection ~ 6250 2800
-Wire Wire Line
-	6050 3100 6250 3100
-Connection ~ 6250 3100
-Wire Wire Line
-	6050 3550 6250 3550
-Connection ~ 6250 3550
-Wire Wire Line
-	6050 3850 6250 3850
-Connection ~ 6250 3850
 $Comp
 L Device:R R1
@@
 	0    1    1    0
 $EndComp
-$Comp
-L Device:R R2
-U 1 1 648FEF5A
-P 5100 1950
-F 0 "R2" V 4893 1950 50  0000 C CNN
-F 1 "R" V 4984 1950 50  0000 C CNN
-F 2 "" V 5030 1950 50  0001 C CNN
-F 3 "~" H 5100 1950 50  0001 C CNN
-	1    5100 1950
-	0    1    1    0
-$EndComp
-$Comp
-L Device:R R3
-U 1 1 648FF522
-P 5100 2700
-F 0 "R3" V 5307 2700 50  0000 C CNN
-F 1 "R" V 5216 2700 50  0000 C CNN
-F 2 "" V 5030 2700 50  0001 C CNN
-F 3 "~" H 5100 2700 50  0001 C CNN
-	1    5100 2700
-	0    -1   -1   0
-$EndComp
-$Comp
-L Device:R R4
-U 1 1 648FF8E0
-P 5100 3450
-F 0 "R4" V 4893 3450 50  0000 C CNN
-F 1 "R" V 4984 3450 50  0000 C CNN
-F 2 "" V 5030 3450 50  0001 C CNN
-F 3 "~" H 5100 3450 50  0001 C CNN
-	1    5100 3450
-	0    1    1    0
-$EndComp
