File: KiCad/24V_to_GPIO/24V_to_GPIO.kicad_sch (KiCad schematic)
At the start: 12 parts, among them U1 4N28

Commit message: Schematics GPIO_to_230V
Parts:
- gave numbers to parts that had none: 2
Connections:
- net +5V: now also R2.1; no longer R2.2
- net Out-1: now also R2.2; no longer R2.1
Other:
- moved on the sheet: R2
Changed lines of the file:
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@@
   (junction (at 82.55 110.49) (diameter 0) (color 0 0 0 0)
   )
+  (junction (at 162.56 33.02) (diameter 0) (color 0 0 0 0)
+  )
   (junction (at 82.55 30.48) (diameter 0) (color 0 0 0 0)
   )
-  (junction (at 162.56 33.02) (diameter 0) (color 0 0 0 0)
-  )
   (wire (pts (xy 153.67 33.02) (xy 162.56 33.02))
     (stroke (width 0) (type default))
@@
     (stroke (width 0) (type default))
   )
+  (wire (pts (xy 162.56 33.02) (xy 166.37 33.02))
+    (stroke (width 0) (type default))
+  )
   (wire (pts (xy 49.53 62.23) (xy 52.07 62.23))
     (stroke (width 0) (type default))
@@
   )
   (wire (pts (xy 80.01 30.48) (xy 82.55 30.48))
-    (stroke (width 0) (type default))
-  )
-  (wire (pts (xy 162.56 33.02) (xy 166.37 33.02))
     (stroke (width 0) (type default))
   )
@@
     )
   )
-  (symbol (lib_id "Device:R") (at 162.56 29.21 180) (unit 1)
-    (in_bom yes) (on_board yes) (dnp no)
-    (property "Reference" "R?" (at 167.8178 29.21 90)
-      (effects (font (size 1.27 1.27)))
-    )
-    (property "Value" "R" (at 165.5064 29.21 90)
-      (effects (font (size 1.27 1.27)))
-    )
-    (property "Footprint" "" (at 164.338 29.21 90)
+  (symbol (lib_id "Device:R") (at 162.56 29.21 0) (unit 1)
+    (in_bom yes) (on_board yes) (dnp no)
+    (property "Reference" "R2" (at 160.2486 29.21 90)
+      (effects (font (size 1.27 1.27)))
+    )
+    (property "Value" "R" (at 162.56 29.21 90)
+      (effects (font (size 1.27 1.27)))
+    )
+    (property "Footprint" "" (at 160.782 29.21 90)
       (effects (font (size 1.27 1.27)) hide)
     )
@@
       (project "24V_to_GPIO"
         (path "/41b01276-b072-4790-9d57-567f16f4294e"
-          (reference "R?") (unit 1)
+          (reference "R2") (unit 1)
         )
       )
@@
   (symbol (lib_id "Device:R_Pack04_SIP_Split") (at 82.55 26.67 0) (unit 1)
     (in_bom yes) (on_board yes) (dnp no)
-    (property "Reference" "RN?" (at 84.7852 25.5016 0)
+    (property "Reference" "RN2" (at 84.7852 25.5016 0)
       (effects (font (size 1.27 1.27)) (justify left))
     )
@@
       (project "24V_to_GPIO"
         (path "/41b01276-b072-4790-9d57-567f16f4294e"
-          (reference "RN?") (unit 1)
+          (reference "RN2") (unit 1)
         )
       )
@@
   (symbol (lib_id "Device:R_Pack04_SIP_Split") (at 82.55 53.34 0) (unit 2)
     (in_bom yes) (on_board yes) (dnp no)
-    (property "Reference" "RN?" (at 84.7852 52.1716 0)
+    (property "Reference" "RN2" (at 84.7852 52.1716 0)
       (effects (font (size 1.27 1.27)) (justify left))
     )
@@
       (project "24V_to_GPIO"
         (path "/41b01276-b072-4790-9d57-567f16f4294e"
-          (reference "RN?") (unit 2)
+          (reference "RN2") (unit 2)
         )
       )
@@
   (symbol (lib_id "Device:R_Pack04_SIP_Split") (at 82.55 80.01 0) (unit 3)
     (in_bom yes) (on_board yes) (dnp no)
-    (property "Reference" "RN?" (at 84.7852 78.8416 0)
+    (property "Reference" "RN2" (at 84.7852 78.8416 0)
       (effects (font (size 1.27 1.27)) (justify left))
     )
@@
       (project "24V_to_GPIO"
         (path "/41b01276-b072-4790-9d57-567f16f4294e"
-          (reference "RN?") (unit 3)
+          (reference "RN2") (unit 3)
         )
       )
@@
   (symbol (lib_id "Device:R_Pack04_SIP_Split") (at 82.55 106.68 0) (unit 4)
     (in_bom yes) (on_board yes) (dnp no)
-    (property "Reference" "RN?" (at 84.7852 105.5116 0)
+    (property "Reference" "RN2" (at 84.7852 105.5116 0)
       (effects (font (size 1.27 1.27)) (justify left))
     )
@@
       (project "24V_to_GPIO"
         (path "/41b01276-b072-4790-9d57-567f16f4294e"
-          (reference "RN?") (unit 4)
+          (reference "RN2") (unit 4)
         )
       )
@@
   (symbol (lib_id "Device:R") (at 134.62 35.56 270) (unit 1)
     (in_bom yes) (on_board yes) (dnp no)
-    (property "Reference" "R1" (at 134.62 30.3022 90)
-      (effects (font (size 1.27 1.27)))
-    )
-    (property "Value" "R" (at 134.62 32.6136 90)
-      (effects (font (size 1.27 1.27)))
-    )
+    (property "Reference" "R1" (at 134.62 33.2486 90)
+      (effects (font (size 1.27 1.27)))
+    )
+    (property "Value" "R" (at 134.62 35.56 90)
+      (effects (font (size 1.27 1.27)))
+    )
