File: KiCad/24V_to_GPIO/24V_to_GPIO.kicad_sch (KiCad schematic)
At the start: 9 parts, among them U1 4N28

Commit message: schematics update
Connections:
- net Out-1 renamed GPIO
- net GPIO: no longer RN2.1 (R1.1), U?.16
- net Out-2 renamed GPIO-2
- net Out-3 renamed GPIO-3
- net Out-4 renamed GPIO-4
- new net GPIO-1: RN2.1 (R1.1), U?.16
Changed lines of the file:
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@@
     )
   )
-  (global_label "Out-4" (shape output) (at 100.33 132.08 0)
+  (global_label "GPIO-4" (shape output) (at 100.33 132.08 0)
     (effects (font (size 1.27 1.27)) (justify left))
     (property "Intersheetrefs" "${INTERSHEET_REFS}" (at 100.33 132.08 0)
@@
     )
   )
-  (global_label "Out-2" (shape output) (at 100.33 78.74 0)
+  (global_label "GPIO-2" (shape output) (at 100.33 78.74 0)
     (effects (font (size 1.27 1.27)) (justify left))
     (property "Intersheetrefs" "${INTERSHEET_REFS}" (at 100.33 78.74 0)
@@
     )
   )
-  (global_label "Out-1" (shape output) (at 181.61 54.61 0)
+  (global_label "GPIO" (shape output) (at 181.61 54.61 0)
     (effects (font (size 1.27 1.27)) (justify left))
     (property "Intersheetrefs" "${INTERSHEET_REFS}" (at 181.61 54.61 0)
@@
     )
   )
-  (global_label "Out-3" (shape output) (at 100.33 105.41 0)
+  (global_label "GPIO-3" (shape output) (at 100.33 105.41 0)
     (effects (font (size 1.27 1.27)) (justify left))
     (property "Intersheetrefs" "${INTERSHEET_REFS}" (at 100.33 105.41 0)
@@
     )
   )
-  (global_label "Out-1" (shape output) (at 100.33 52.07 0)
+  (global_label "GPIO-1" (shape output) (at 100.33 52.07 0)
     (effects (font (size 1.27 1.27)) (justify left))
     (property "Intersheetrefs" "${INTERSHEET_REFS}" (at 100.33 52.07 0)
